Commit message: changes

File: husky_commander/config/husky_basic/robot.urdf.xacro (robot description, xacro)
@@ -16,10 +16,43 @@
   </xacro:bumper>
   <xacro:include filename="$(find clearpath_platform_description)/urdf/a200/attachments/top_plate.urdf.xacro"/>
-  <xacro:top_plate name="top_plate" model="default" parent_link="default_mount">
+  <xacro:top_plate name="top_plate" model="pacs" parent_link="default_mount">
     <origin xyz="0.0 0.0 0.0" rpy="0.0 0.0 0.0"/>
   </xacro:top_plate>
+  <xacro:include filename="$(find clearpath_platform_description)/urdf/a200/attachments/sensor_arch.urdf.xacro"/>
+  <xacro:sensor_arch name="sensor_arch" model="sensor_arch_300" parent_link="default_mount">
+    <origin xyz="0.0 0.0 0.0" rpy="0.0 0.0 0.0"/>
+  </xacro:sensor_arch>
   <!-- Links -->
+  <xacro:include filename="$(find clearpath_platform_description)/urdf/links/box.urdf.xacro"/>
+  <xacro:box name="user_bay_cover" parent_link="top_plate_link" size="0.4 0.4 0.002">
+    <origin xyz="0.0 0.0 0.00735" rpy="0.0 0.0 0.0"/>
+  </xacro:box>
   <!-- Mounts -->
+  <!-- fath_pivot_0 -->
+  <xacro:include filename="$(find clearpath_mounts_description)/urdf/fath_pivot.urdf.xacro"/>
+  <xacro:fath_pivot name="fath_pivot_0" parent_link="sensor_arch_mount" angle="0.0">
+    <origin xyz="0.0 0.0 -0.021" rpy="3.1415 0.0 0.0"/>
+  </xacro:fath_pivot>
+  <!-- bracket_0 -->
+  <xacro:include filename="$(find clearpath_mounts_description)/urdf/pacs/bracket.urdf.xacro"/>
+  <xacro:bracket name="bracket_0" parent_link="top_plate_mount_d1" model="horizontal">
+    <origin xyz="0.0 0.0 0.0" rpy="0.0 0.0 0.0"/>
+  </xacro:bracket>
   <!-- Sensors -->
+  <!-- lidar2d_0 -->
+  <xacro:include filename="$(find clearpath_sensors_description)/urdf/hokuyo_ust.urdf.xacro"/>
+  <xacro:hokuyo_ust name="lidar2d_0" parent_link="bracket_0_mount" ang_res="0.5" min_ang="-2.356" max_ang="2.356" min_range="0.05" max_range="25.0" update_rate="50">
+    <origin xyz="0.0 0.0 0.0" rpy="0.0 0.0 0.0"/>
+  </xacro:hokuyo_ust>
+  <!-- lidar3d_0 -->
+  <xacro:include filename="$(find clearpath_sensors_description)/urdf/velodyne_lidar.urdf.xacro"/>
+  <xacro:velodyne_lidar name="lidar3d_0" parent_link="sensor_arch_mount" ang_res_h="0.4" ang_res_v="2.0" min_ang_h="-3.141592" max_ang_h="3.141592" min_ang_v="-0.261799" max_ang_v="0.261799" min_range="0.9" max_range="130.0" update_rate="50">
+    <origin xyz="0.0 0.0 0.0" rpy="0.0 0.0 0.0"/>
+  </xacro:velodyne_lidar>
+  <!-- camera_0 -->
+  <xacro:include filename="$(find clearpath_sensors_description)/urdf/intel_realsense.urdf.xacro"/>
+  <xacro:intel_realsense name="camera_0" parent_link="fath_pivot_0_mount" update_rate="30" image_height="480" image_width="640">
+    <origin xyz="0.0 0.0 0.0" rpy="0.0 0.0 0.0"/>
+  </xacro:intel_realsense>
   <!-- Manipulators -->
   <!-- Extras -->
